Commit message: experiment final

File: experiment_03/urdf/arm_urdf.urdf (robot description, URDF)
Before this commit: robot simple_manipulator, 5 links, 4 joints
Links:
- removed link link_base
- added link base_link, mass 5; collision cylinder length=0.04 radius=0.1; visual cylinder length=0.04 radius=0.1
Joints:
- joint base_footprint_joint: child link_base -> base_link
- joint link_1_joint: parent link_base -> base_link
